File: Receiver Schematic.kicad_pcb (KiCad board)
At the start: 2 copper layers, 31 parts

Commit message: First version with a pcb
V3
Parts:
- removed 0.1uF (x6), 1000 (x2), 130pF (x2), 14pF (x2), 2.2nF, 22nF (x2): C_0805_2012Metric, Capacitor_SMD:C_0805_2012Metric
- removed 160 (x2), 51K (x2): R_0805_2012Metric, Capacitor_SMD:C_0805_2012Metric
- removed 180nH, 2.7uH (x2): L_0805_2012Metric, Inductor_SMD:L_0805_2012Metric
- removed 51 (x4): R_2512_6332Metric, Resistor_SMD:R_2512_6332Metric
- removed 7.5nF (x2): C_1206_3216Metric, Capacitor_SMD:C_1206_3216Metric
- removed AD8041 (x2): SOIC-8-1EP_3.9x4.9mm_P1.27mm_EP2.29x3mm, Package_SO:SOIC-8-1EP_3.9x4.9mm_P1.27mm_EP2.29x3mm
- removed Crystal_GND24_Small: MSOP-10_3x3mm_P0.5mm, Package_SO:MSOP-10_3x3mm_P0.5mm
- added AntennaConnector1: Conn_Coaxial, Connector_Coaxial:BNC_Amphenol_B6252HB-NPP3G-50_Horizontal, F.Cu at (85.4, 127.6)
- added C10: 10uF, lmao:CAP_EEEFK1C100R, F.Cu at (111.8, 48.9)
- added C11: 0.1u, Capacitor_SMD:C_0805_2012Metric, F.Cu at (112.1, 97.2)
- added C12: 0.1u, Capacitor_SMD:C_0805_2012Metric, F.Cu at (66.7, 111.1)
- added C13: 0.1u, Capacitor_SMD:C_0805_2012Metric, F.Cu at (119.4, 101.2)
- added C14: 7.5n, Capacitor_SMD:C_1206_3216Metric, F.Cu at (114.3, 74.9)
- added C15: 22n, Capacitor_SMD:C_0805_2012Metric, F.Cu at (128.9, 74.9)
- added C16: 14p, Capacitor_SMD:C_0805_2012Metric, F.Cu at (137.2, 65.4)
- added C17: 14p, Capacitor_SMD:C_0805_2012Metric, F.Cu at (121.9, 64.8)
- added C18: 0.1u, Capacitor_SMD:C_0805_2012Metric, F.Cu at (130.2, 65.1)
- added C19: 10uF, Capacitor_SMD:C_0805_2012Metric, F.Cu at (142.2, 62.2)
- added C2: 0.1u, Capacitor_SMD:C_0805_2012Metric, F.Cu at (56.5, 66.0)
- added C20: 10uF, Capacitor_SMD:C_0805_2012Metric, F.Cu at (124.5, 60.6)
- added C3: 130pF, Capacitor_SMD:C_0805_2012Metric, F.Cu at (98.4, 130.2)
- added C4: 10nF, Capacitor_SMD:C_0805_2012Metric, F.Cu at (111.8, 59.1)
- added C5: 2.2nF, Capacitor_SMD:C_0805_2012Metric, F.Cu at (108.0, 127.0)
- added C6: 100nF, Capacitor_SMD:C_0805_2012Metric, F.Cu at (111.8, 54.0)
- added C7: 130pF, Capacitor_SMD:C_0805_2012Metric, F.Cu at (116.8, 130.2)
- added C8: 22n, Capacitor_SMD:C_0805_2012Metric, F.Cu at (143.5, 73.7)
- added C9: 7.5n, Capacitor_SMD:C_1206_3216Metric, F.Cu at (143.5, 79.4)
- added J1: AudioJack3, Connector_Audio:Jack_3.5mm_CUI_SJ-3523-SMT_Horizontal, F.Cu at (133.3, 54.0)
- added J2: USB_A, Connector_USB:USB_A_Molex_67643_Horizontal, F.Cu at (104.5, 58.7)
- added L1: 2.7uH, Capacitor_SMD:C_0805_2012Metric, F.Cu at (103.5, 130.2)
- added L2: 180nH, Capacitor_SMD:C_0805_2012Metric, F.Cu at (112.4, 127.0)
- added L3: 2.7uH, Capacitor_SMD:C_0805_2012Metric, F.Cu at (121.9, 130.2)
- added R1: 1000, Resistor_SMD:R_0805_2012Metric, F.Cu at (113.0, 101.2)
- added R10: 160, Resistor_SMD:R_0805_2012Metric, F.Cu at (121.9, 74.9)
- added R11: 4.7k, Resistor_SMD:R_0805_2012Metric, F.Cu at (64.1, 101.0)
- added R12: 4.7k, Resistor_SMD:R_0805_2012Metric, F.Cu at (64.1, 107.3)
- added R2: 1000, Resistor_SMD:R_0805_2012Metric, F.Cu at (113.0, 105.4)
- added R3: 51, Resistor_SMD:R_2512_6332Metric, F.Cu at (132.1, 87.0)
- added R4: 51, Resistor_SMD:R_2512_6332Metric, F.Cu at (140.3, 87.0)
- added R5: 51, Resistor_SMD:R_2512_6332Metric, F.Cu at (117.5, 87.0)
- added R6: 51, Resistor_SMD:R_2512_6332Metric, F.Cu at (124.5, 87.0)
- added R7: 51k, Resistor_SMD:R_0805_2012Metric, F.Cu at (128.9, 71.1)
- added R8: 51k, Resistor_SMD:R_0805_2012Metric, F.Cu at (143.5, 69.8)
- added R9: 160, Resistor_SMD:R_0805_2012Metric, F.Cu at (136.9, 74.9)
- added TP1: TestPoint, TestPoint:TestPoint_THTPad_2.0x2.0mm_Drill1.0mm, F.Cu at (93.3, 134.0)
- added TP10: TestPoint, TestPoint:TestPoint_THTPad_2.0x2.0mm_Drill1.0mm, F.Cu at (115.6, 69.8)
- added TP11: TestPoint, TestPoint:TestPoint_THTPad_2.0x2.0mm_Drill1.0mm, F.Cu at (125.7, 75.6)
- added TP12: TestPoint, TestPoint:TestPoint_THTPad_2.0x2.0mm_Drill1.0mm, F.Cu at (135.9, 84.5)
- added TP13: TestPoint, TestPoint:TestPoint_THTPad_2.0x2.0mm_Drill1.0mm, F.Cu at (140.3, 76.2)
- added TP14: TestPoint, TestPoint:TestPoint_THTPad_2.0x2.0mm_Drill1.0mm, F.Cu at (142.9, 57.1)
- added TP15: TestPoint, TestPoint:TestPoint_THTPad_2.0x2.0mm_Drill1.0mm, F.Cu at (120.0, 59.7)
- added TP2: TestPoint, TestPoint:TestPoint_THTPad_2.0x2.0mm_Drill1.0mm, F.Cu at (83.8, 111.8)
- added TP3: TestPoint, TestPoint:TestPoint_THTPad_2.0x2.0mm_Drill1.0mm, F.Cu at (130.8, 110.5)
- added TP4: TestPoint, TestPoint:TestPoint_THTPad_2.0x2.0mm_Drill1.0mm, F.Cu at (83.8, 102.2)
- added TP5: TestPoint, TestPoint:TestPoint_THTPad_2.0x2.0mm_Drill1.0mm, F.Cu at (83.8, 106.7)
- added TP6: TestPoint, TestPoint:TestPoint_THTPad_2.0x2.0mm_Drill1.0mm, F.Cu at (133.3, 93.5)
- added TP7: TestPoint, TestPoint:TestPoint_THTPad_2.0x2.0mm_Drill1.0mm, F.Cu at (141.6, 93.5)
- added TP8: TestPoint, TestPoint:TestPoint_THTPad_2.0x2.0mm_Drill1.0mm, F.Cu at (116.2, 93.5)
- added TP9: TestPoint, TestPoint:TestPoint_THTPad_2.0x2.0mm_Drill1.0mm, F.Cu at (122.6, 93.5)
- added U1: Pico, MCU_RaspberryPi_and_Boards:RPi_Pico_SMD_TH, F.Cu at (78.1, 84.5)
- added U2: Si5351A-B-GT, Package_SO:MSOP-10_3x3mm_P0.5mm, F.Cu at (75.6, 106.0)
- added U3: SN74CBT3253, Package_SO:SOIC-16_3.9x9.9mm_P1.27mm, F.Cu at (127.6, 103.1)
- added U4: R_8_ADI, AD8041ARZ:AD8041ARZ, F.Cu at (137.2, 69.2)
- added U5: R_8_ADI, AD8041ARZ:AD8041ARZ, F.Cu at (121.9, 69.8)
- added Y1: CX3225SB 25MHz, Crystal:Crystal_SMD_TXC_7M-4Pin_3.2x2.5mm, F.Cu at (75.6, 111.1)
Routing:
- net Smoothed 5V: track 0.00 -> 228.1 mm
- net Net-(L3-Pad2): track 0.00 -> 59.5 mm
- net Net-(TP4-Pad1): track 0.00 -> 52.2 mm
- net Net-(TP5-Pad1): track 0.00 -> 51.1 mm, vias 0 -> 2
- net +3V3: track 0.00 -> 50.7 mm
- net GND: track 0.00 -> 45.4 mm, vias 0 -> 8
- net Net-(AntennaConnector1-Pad2): track 0.00 -> 31.7 mm
- net /180 degrees: track 0.00 -> 28.5 mm, vias 0 -> 2
- net Net-(C9-Pad1): track 0.00 -> 27.9 mm
- net /270 degrees: track 0.00 -> 27.3 mm
- net /SCL: track 0.00 -> 26.1 mm, vias 0 -> 2
- net Net-(C16-Pad1): track 0.00 -> 24.2 mm
- net Net-(C8-Pad1): track 0.00 -> 22.5 mm, vias 0 -> 2
- net /90 degrees: track 0.00 -> 22.3 mm
- net Net-(C15-Pad2): track 0.00 -> 21.3 mm
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- added copper zone on B.Cu, net GND
- added copper zone on F.Cu, net GND
Other:
- board outline added: 95.3 x 95.2 mm
- board text added: "3rd Order BandPass Filter 7-12MHZ"
- board text added: "DC Offset"
- board text added: "Multiple Feedback Low Pass Amplifier 1000 V/V 1000kHz"
- board text added: "Oscillator 25MHz"
- board text added: "Raspberry Pi Pico"
- board text added: "Tayloe Mixer"
- board text added: "USB A Input"
- board text added: "Voltage Smoother"

Commit message: V4
V4
Parts:
- removed C2: 0.1u, Capacitor_SMD:C_0805_2012Metric
- removed J2: USB_A, Connector_USB:USB_A_Molex_67643_Horizontal
- removed U5: R_8_ADI, AD8041ARZ:AD8041ARZ
- added R13: 1, Resistor_SMD:R_0805_2012Metric, F.Cu at (81.3, 55.4)
- C10: value 10uF -> 8200uF; footprint lmao:CAP_EEEFK1C100R -> Capacitor_THT:CP_Radial_D16.0mm_P7.50mm
- C9: footprint Capacitor_SMD:C_1206_3216Metric -> Capacitor_SMD:C_0805_2012Metric
- J1: value AudioJack3 -> SJ1-3525N; footprint Connector_Audio:Jack_3.5mm_CUI_SJ-3523-SMT_Horizontal -> CUI_SJ1-3225N:CUI_SJ1-3525N
- L1, L2, L3: footprint Capacitor_SMD:C_0805_2012Metric -> Inductor_THT:L_Toroid_Vertical_L10.0mm_W5.0mm_P5.08mm
- R3, R4, R5, R6: footprint Resistor_SMD:R_2512_6332Metric -> Resistor_SMD:R_0805_2012Metric
- U4: value R_8_ADI -> LM2904; footprint AD8041ARZ:AD8041ARZ -> Package_SO:SOIC-8_3.9x4.9mm_P1.27mm
- moved C4 23.5 mm to (88.4, 56.4), turned to -90 degrees
- moved AntennaConnector1 21.6 mm to (63.8, 128.3)
- moved C6 17.9 mm to (94.0, 56.4), turned to -90 degrees
- moved C10 10.6 mm to (106.2, 57.9), turned to 90 degrees
- moved L3 7.11 mm to (129.0, 130.0), turned to 90 degrees
- moved C7 7.11 mm to (124.0, 130.2)
- moved U4 6.25 mm to (131.1, 70.6), turned to 0 degrees
- moved L2 6.05 mm to (118.4, 126.0), turned to 180 degrees
- moved C15 5.66 mm to (125.0, 70.9)
- moved R7 5.66 mm to (125.0, 67.1)
- moved C5 3.82 mm to (110.7, 124.4)
- moved TP12 3.43 mm to (135.9, 87.9)
- moved J1 2.95 mm to (132.1, 51.3), turned to -90 degrees
- moved R3 2.03 mm to (132.1, 89.0)
- moved R4 2.03 mm to (140.3, 89.0)
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Connections:
- U1 pad 39: Smoothed 5V -> unconnected-(U1-Pad39)
- U1 pad 40: Smoothed 5V -> 5V
- U4 pad 1: unconnected-(U4-Pad1) -> Net-(C16-Pad1)
- U4 pad 5: unconnected-(U4-Pad5) -> Net-(C14-Pad2)
- U4 pad 6: Net-(C16-Pad1) -> Net-(C17-Pad1)
- U4 pad 7: Smoothed 5V -> Net-(C17-Pad2)
- U4 pad 8: unconnected-(U4-Pad8) -> Smoothed 5V
Routing:
- net Smoothed 5V: track 228.1 -> 129.5 mm
- net 5V: track 0.00 -> 42.2 mm
- net GND: track 45.4 -> 23.2 mm, vias 8 -> 6
- net Net-(AntennaConnector1-Pad2): track 31.7 -> 51.9 mm
- net Net-(C14-Pad2): track 21.0 -> 38.9 mm, vias 0 -> 2
- net Net-(C17-Pad1): track 15.4 -> 31.4 mm, vias 0 -> 4
- net unconnected-(J2-Pad5): track 13.1 -> 0.00 mm
- net Net-(C5-Pad1): track 15.9 -> 24.1 mm
- net Net-(L3-Pad2): track 59.5 -> 52.8 mm
- net Net-(C16-Pad2): track 16.0 -> 21.1 mm
- net Net-(C16-Pad1): track 24.2 -> 29.0 mm, vias 0 -> 2
- net Net-(C9-Pad1): track 27.9 -> 32.5 mm
- net Net-(C8-Pad1): track 22.5 -> 25.8 mm, vias 2 -> 4
- net /Q signal: track 7.38 -> 4.47 mm
- net Net-(C17-Pad2): track 20.5 -> 21.9 mm
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Other:
- board text added: "Cadyn Maddocks & Taylor Smith SDR Receiver Project Electronics II V4"
- board text added: "DC Offset 2.5V"
- board text removed: "DC Offset"
