File: Receiver Schematic.kicad_sch (KiCad schematic)
At the start: 57 parts, among them J1 AudioJack3, U1 Pico, U2 Si5351A-B-GT, U3 SN74CBT3253, U4 LT6231CDD#PBF, U5 LT6231CDD#PBF, Y1 Crystal_GND24_Small

Commit message: V2
Parts:
- removed C1: 510p, symbol Device:C_Small
- removed C10, C11: 7.5n, symbol Device:C_Small
- removed C12, C13: 16pF, symbol Device:C_Small
- removed C2, C4, C6: 5.6n, symbol Device:C_Small
- removed C?: (no value), symbol Device:C_Small
- removed TP10, TP11, TP13, TP8, TP9: TestPoint, symbol Connector:TestPoint
- added C14: 7.5n, symbol Device:C_Small
- added C15: 22n, symbol Device:C_Small
- added C16, C17: 14p, symbol Device:C_Small
- added C?: (no value), symbol Device:C_Polarized_Small_US
- added R10, R9: 160, symbol Device:R_Small_US
- C3: value 180p -> 130pF
- C4, C6: renamed from C?; value (none) -> C_Small
- C5: value 180p -> 2.2nF
- C7: value 510p -> 130pF
- C8: value 7.5n -> 22n
- J2: renamed from J?; value (none) -> USB_A
- L1, L3: value 82n -> 2.7uH
- L2: value 82n -> 180nH
- R7, R8: value 100k -> 51k
- Y1: value Crystal_GND24_Small -> (none)
- gave numbers to parts that had none: 6
Connections:
- net +5V: no longer C11.2, C13.2, C18.2, C4.1, C6.1, J2.1 (VBUS), R1.1, U3.16 (VCC), U4.7 (V+), U5.7 (V+)
- net 270 degrees: now also R5.1; no longer R6.1
- net 90 degrees: now also R6.1; no longer R5.1
- net GND: now also C5.2, C14.1, C15.1, C?.2; no longer L1.2, L3.2
- net I signal: now also R8.2, C16.1; no longer R7.2
- net Q signal: now also R7.2, C17.2; no longer R8.2
- net at R1.2, R2.1, TP3.1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: now also L3.2; no longer C7.2
- net SCL: now reaches U1.7 (GPIO5), U2.4 (SCL)
- net SDA: now reaches U1.6 (GPIO4), U2.5 (SDA)
- net at C8.1, R3.2: now also R8.1, R9.1; no longer R7.1, U4.2 (-)
- net at AntennaConnector1.2 (Ext), TP1.1: now also C3.2
- net at C5.1, L2.1: now also C7.1, L1.2; no longer C3.2
- net at U5.3 (+): now also R5.2, C14.2; no longer R6.2
- new net: C7.2, L3.1
- new net: C15.2, R10.1, R6.2, R7.1
- new net: C17.1, R10.2, U5.2 (-)
- new net: C16.2, R9.2, U4.2 (-)
- new net Smoothed 5V: C11.2, C13.2, C18.2, C4.1, C6.1, C?.1, J2.1 (VBUS), R1.1, U3.16 (VCC), U4.7 (V+), U5.7 (V+)
- no-connect marks 0 -> 41
Other:
- note added: "7-12Mhz BandPass Filter"

Commit message: First version with a pcb
V3
Parts:
- removed C1: 0.1u, symbol Device:C_Small
- added C19, C20: 10uF, Capacitor_SMD:C_0805_2012Metric, symbol Device:C_Small
- added R11, R12: 4.7k, Resistor_SMD:R_0805_2012Metric, symbol Device:R_Small_US
- added TP10, TP11, TP13, TP8, TP9: TestPoint, TestPoint:TestPoint_THTPad_2.0x2.0mm_Drill1.0mm, symbol Connector:TestPoint
- AntennaConnector1: value Conn_Coaxial -> (none)
- C10: renamed from C?; value (none) -> 10uF; footprint (none) -> lmao:CAP_EEEFK1C100R
- C11, C12, C13, C15, C16, C17, C18, C2, C3, C5, C7, C8, L1, L2, L3: footprint (none) -> Capacitor_SMD:C_0805_2012Metric
- C14, C9: footprint (none) -> Capacitor_SMD:C_1206_3216Metric
- C4: value C_Small -> 10nF; footprint (none) -> Capacitor_SMD:C_0805_2012Metric
- C6: value C_Small -> 100nF; footprint (none) -> Capacitor_SMD:C_0805_2012Metric
- J1: footprint (none) -> Connector_Audio:Jack_3.5mm_CUI_SJ-3523-SMT_Horizontal
- J2: footprint (none) -> Connector_USB:USB_A_Molex_67643_Horizontal
- R1, R10, R2, R7, R8, R9: footprint (none) -> Resistor_SMD:R_0805_2012Metric
- R3, R4, R5, R6: footprint (none) -> Resistor_SMD:R_2512_6332Metric
- TP1, TP12, TP14, TP15, TP2, TP3, TP4, TP5, TP6, TP7: footprint (none) -> TestPoint:TestPoint_THTPad_2.0x2.0mm_Drill1.0mm
- U1: footprint RPi_Pico:RPi_Pico_SMD_TH -> MCU_RaspberryPi_and_Boards:RPi_Pico_SMD_TH
- U3: footprint (none) -> Package_SO:SOIC-16_3.9x9.9mm_P1.27mm
- U4, U5: value LT6231CDD#PBF -> AD8041ARZ; footprint Package_SO:SOIC-8_3.9x4.9mm_P1.27mm -> AD8041ARZ:AD8041ARZ
- Y1: value (none) -> CX3225SB 25MHz; footprint (none) -> Crystal:Crystal_SMD_TXC_7M-4Pin_3.2x2.5mm
Connections:
- net +5V is gone; now on net Smoothed 5V: C2.1, U1.40 (VBUS)
- net +3V3: now also U1.36 (3V3), R11.2, R12.2; no longer U1.39 (VSYS)
- net 270 degrees: now also TP8.1
- net 90 degrees: now also TP9.1
- net I signal: now also C19.2; no longer C16.1, R8.2, TP14.1, U4.6
- net Q signal: now also C20.2; no longer C17.2, R7.2, TP15.1, U5.6
- net SCL: now also R12.1
- net SDA: now also R11.1
- net Smoothed 5V: now also U1.39 (VSYS)
- net at C14.2, R5.2, U5.3 (+): now also TP10.1
- net at C17.1, R10.2, U5.2 (-): now also TP11.1
- net at C16.2, R9.2, U4.2 (-): now also TP13.1
- new net: C17.2, C20.1, R7.2, TP15.1, U5.6
- new net: C16.1, C19.1, R8.2, TP14.1, U4.6
- no-connect marks 41 -> 40

Commit message: V4
V4
Parts:
- removed C2: 0.1u, Capacitor_SMD:C_0805_2012Metric, symbol Device:C_Small
- removed J1: AudioJack3, Connector_Audio:Jack_3.5mm_CUI_SJ-3523-SMT_Horizontal, symbol Connector:AudioJack3
- removed J2: USB_A, Connector_USB:USB_A_Molex_67643_Horizontal, symbol Connector:USB_A
- removed U4, U5: AD8041ARZ, AD8041ARZ:AD8041ARZ, symbol Amplifier_Operational:OPA333xxD
- added J1: SJ1-3525N, CUI_SJ1-3225N:CUI_SJ1-3525N, symbol Audio_Jack_Sterio3:SJ1-3525N
- added R13: 1, Resistor_SMD:R_0805_2012Metric, symbol Device:R_Small_US
- added U4: LM2904, Package_SO:SOIC-8_3.9x4.9mm_P1.27mm, symbol Amplifier_Operational:LM2904
- AntennaConnector1: value (none) -> Conn_Coaxial; footprint (none) -> Connector_Coaxial:BNC_Amphenol_B6252HB-NPP3G-50_Horizontal
- C10: value 10uF -> 8200uF; footprint lmao:CAP_EEEFK1C100R -> Capacitor_THT:CP_Radial_D16.0mm_P7.50mm
- C9: footprint Capacitor_SMD:C_1206_3216Metric -> Capacitor_SMD:C_0805_2012Metric
- L1, L2, L3: footprint Capacitor_SMD:C_0805_2012Metric -> Inductor_THT:L_Toroid_Vertical_L10.0mm_W5.0mm_P5.08mm
- R3, R4, R5, R6: footprint Resistor_SMD:R_2512_6332Metric -> Resistor_SMD:R_0805_2012Metric
Connections:
- net GND: now also J1.1, U4.4 (V-)
- net I signal: now also J1.3
- net Q signal: now also J1.2
- net Smoothed 5V: now also R13.2, U4.8 (V+); no longer U1.39 (VSYS), U1.40 (VBUS)
- net at C17.1, R10.2, TP11.1: now also U4.6 (-)
- net at C14.2, R5.2, TP10.1: now also U4.5 (+)
- net at C9.1, R4.2, TP12.1: now also U4.3 (+)
- net at C17.2, C20.1, R7.2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: now also U4.7
- net at C16.1, C19.1, R8.2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: now also U4.1
- net at C16.2, R9.2, TP13.1: now also U4.2 (-)
- new net 5V: R13.1, U1.40 (VBUS)
Other:
- note added: "Cadyn Maddocks & Taylor Smith SDR Receiver Electronics II V4"
- note added: "DC Blocking Capacitors"
- note added: "Lm2904 Power Supply"
- note added: "Multiple Feedback Lowpass Filter & Amplifier 1000 V/V with Cutoff Frequency of approx 100kHz"
- note added: "Oscillator"
- note added: "Tayloe Mixer"
- note added: "Voltage Smoother"
- title: (none) -> SDR Receiver
- moved on the sheet: C18, C19, C20, TP3
