File: Kicad Schematic V5/Receiver Schematic.kicad_sch (KiCad schematic)
At the start: 56 parts, among them J1 SJ1-3525N, U1 Pico, U2 Si5351A-B-GT, U3 SN74CBT3253, U4 LM2904, Y1 CX3225SB 25MHz

Commit message: Version 5
Updated File organization and minor fixes.
Parts:
- C14: footprint Capacitor_SMD:C_1206_3216Metric -> Capacitor_SMD:C_0805_2012Metric
- U4: value LM2904 -> LM4562MA
Connections:
- net GND: now also AntennaConnector1.2 (Ext); no longer AntennaConnector1.1 (In)
- net at C3.2, TP1.1: now also AntennaConnector1.1 (In); no longer AntennaConnector1.2 (Ext)
Other:
- note added: "LM4562MA Power Supply"
- note removed: "Lm2904 Power Supply"
- moved on the sheet: AntennaConnector1
Changed lines of the file:
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@@
     (effects (font (size 1.27 1.27)) (justify left bottom))
   )
-  (text "Lm2904 Power Supply" (at 180.34 91.44 0)
+  (text "LM4562MA Power Supply" (at 180.34 91.44 0)
     (effects (font (size 1.27 1.27)) (justify left bottom))
   )
@@
       (effects (font (size 1.27 1.27)) (justify left))
     )
-    (property "Footprint" "Capacitor_SMD:C_1206_3216Metric" (id 2) (at 186.69 58.42 0)
+    (property "Footprint" "Capacitor_SMD:C_0805_2012Metric" (id 2) (at 186.69 58.42 0)
       (effects (font (size 1.27 1.27)) hide)
     )
@@
     (pin "1")
   )
-  (symbol (lib_id "Connector:Conn_Coaxial") (at 17.78 57.15 90) (unit 1)
-    (in_bom yes) (on_board yes) (fields_autoplaced)
-    (property "Reference" "AntennaConnector1" (id 0) (at 18.0732 49.53 90))
-    (property "Value" "Conn_Coaxial" (id 1) (at 18.0732 52.07 90))
+  (symbol (lib_id "Connector:Conn_Coaxial") (at 17.78 57.15 0) (mirror y) (unit 1)
+    (in_bom yes) (on_board yes) (fields_autoplaced)
+    (property "Reference" "AntennaConnector1" (id 0) (at 18.0974 49.53 0))
+    (property "Value" "Conn_Coaxial" (id 1) (at 18.0974 52.07 0))
     (property "Footprint" "Connector_Coaxial:BNC_Amphenol_B6252HB-NPP3G-50_Horizontal" (id 2) (at 17.78 57.15 0)
       (effects (font (size 1.27 1.27)) hide)
@@
     (in_bom yes) (on_board yes) (fields_autoplaced)
     (property "Reference" "U4" (id 0) (at 217.17 31.75 0))
-    (property "Value" "LM2904" (id 1) (at 217.17 34.29 0))
+    (property "Value" "LM4562MA" (id 1) (at 217.17 34.29 0))
     (property "Footprint" "Package_SO:SOIC-8_3.9x4.9mm_P1.27mm" (id 2) (at 217.17 41.91 0)
       (effects (font (size 1.27 1.27)) hide)
     )
-    (property "Datasheet" "http://www.ti.com/lit/ds/symlink/lm358.pdf" (id 3) (at 217.17 41.91 0)
+    (property "Datasheet" "https://www.ti.com/lit/ds/snas326k/snas326k.pdf" (id 3) (at 217.17 41.91 0)
       (effects (font (size 1.27 1.27)) hide)
     )
@@
     (in_bom yes) (on_board yes) (fields_autoplaced)
     (property "Reference" "U4" (id 0) (at 217.17 54.61 0))
-    (property "Value" "LM2904" (id 1) (at 217.17 57.15 0))
+    (property "Value" "LM4562MA" (id 1) (at 217.17 57.15 0))
     (property "Footprint" "Package_SO:SOIC-8_3.9x4.9mm_P1.27mm" (id 2) (at 217.17 64.77 0)
       (effects (font (size 1.27 1.27)) hide)
     )
-    (property "Datasheet" "http://www.ti.com/lit/ds/symlink/lm358.pdf" (id 3) (at 217.17 64.77 0)
+    (property "Datasheet" "https://www.ti.com/lit/ds/snas326k/snas326k.pdf" (id 3) (at 217.17 64.77 0)
       (effects (font (size 1.27 1.27)) hide)
     )
@@
   )
   (symbol (lib_id "Connector:TestPoint") (at 205.74 62.23 0) (unit 1)
-    (in_bom yes) (on_board yes) (fields_autoplaced)
-    (property "Reference" "TP10" (id 0) (at 208.28 57.6579 0)
-      (effects (font (size 1.27 1.27)) (justify left))
-    )
-    (property "Value" "TestPoint" (id 1) (at 208.28 60.1979 0)
+    (in_bom yes) (on_board yes)
+    (property "Reference" "TP10" (id 0) (at 207.01 57.15 0)
+      (effects (font (size 1.27 1.27)) (justify left))
+    )
+    (property "Value" "TestPoint" (id 1) (at 207.01 59.69 0)
       (effects (font (size 1.27 1.27)) (justify left))
     )
@@
       (effects (font (size 1.27 1.27)) (justify left))
     )
-    (property "Value" "LM2904" (id 1) (at 189.23 110.4899 0)
+    (property "Value" "LM4562MA" (id 1) (at 189.23 110.4899 0)
       (effects (font (size 1.27 1.27)) (justify left))
     )
@@
       (effects (font (size 1.27 1.27)) hide)
     )
-    (property "Datasheet" "http://www.ti.com/lit/ds/symlink/lm358.pdf" (id 3) (at 190.5 109.22 0)
+    (property "Datasheet" "https://www.ti.com/lit/ds/snas326k/snas326k.pdf" (id 3) (at 190.5 109.22 0)
       (effects (font (size 1.27 1.27)) hide)
     )
@@
     )
     (path "/113ef254-820a-43ee-81cd-2b01c043d894"
-      (reference "C14") (unit 1) (value "7.5n") (footprint "Capacitor_SMD:C_1206_3216Metric")
+      (reference "C14") (unit 1) (value "7.5n") (footprint "Capacitor_SMD:C_0805_2012Metric")
     )
     (path "/12a4a4ec-1bc7-46d4-a729-c41e56dd799d"
@@
     )
     (path "/3ea84907-c408-45f9-8acd-60f41df45e6f"
-      (reference "U4") (unit 1) (value "LM2904") (footprint "Package_SO:SOIC-8_3.9x4.9mm_P1.27mm")
+      (reference "U4") (unit 1) (value "LM4562MA") (footprint "Package_SO:SOIC-8_3.9x4.9mm_P1.27mm")
     )
     (path "/f4221855-6e91-4693-826c-bfa7fd4d2334"
-      (reference "U4") (unit 2) (value "LM2904") (footprint "Package_SO:SOIC-8_3.9x4.9mm_P1.27mm")
+      (reference "U4") (unit 2) (value "LM4562MA") (footprint "Package_SO:SOIC-8_3.9x4.9mm_P1.27mm")
     )
     (path "/f5266879-01c3-48a4-8f6c-ac9c7c5f9e2e"
-      (reference "U4") (unit 3) (value "LM2904") (footprint "Package_SO:SOIC-8_3.9x4.9mm_P1.27mm")
+      (reference "U4") (unit 3) (value "LM4562MA") (footprint "Package_SO:SOIC-8_3.9x4.9mm_P1.27mm")
     )
     (path "/a64d4d7a-f8d3-4e20-ab2d-06f2152a01cc"
