File: Kicad V6/Receiver Schematic.kicad_pcb (KiCad board)
At the start: 2 copper layers, 95.3 x 95.2 mm, 56 parts, among them J1 SJ1-3525N, U1 Pico, U2 Si5351A-B-GT, U3 SN74CBT3253, U4 LM4562MA, Y1 CX3225SB 25MHz

Commit message: Final Schematic/PCB version
Version 6 of the SDR Design
Parts:
- C14, C9: value 7.5n -> 6.8n
- C16, C17: value 14p -> 1n
- R10, R9: value 160 -> 51
- R7, R8: value 51k -> 5.1k
Connections:
- AntennaConnector1 pad 1: GND -> Net-(AntennaConnector1-Pad1)
- AntennaConnector1 pad 2: Net-(AntennaConnector1-Pad2) -> GND
- C3 pad 2: Net-(AntennaConnector1-Pad2) -> Net-(AntennaConnector1-Pad1)
- TP1 pad 1: Net-(AntennaConnector1-Pad2) -> Net-(AntennaConnector1-Pad1)
Routing:
- net Net-(AntennaConnector1-Pad2): track 51.9 -> 0.00 mm
- net Net-(AntennaConnector1-Pad1): track 0.00 -> 37.6 mm
Other:
- board text added: "Cadyn Maddocks & Taylor Smith SDR Receiver Project Electronics II V6"
- board text removed: "Cadyn Maddocks & Taylor Smith SDR Receiver Project Electronics II V4"
