File: Kicad V6/Receiver Schematic.kicad_sch (KiCad schematic)
At the start: 56 parts, among them J1 SJ1-3525N, U1 Pico, U2 Si5351A-B-GT, U3 SN74CBT3253, U4 LM4562MA, Y1 CX3225SB 25MHz

Commit message: Final Schematic/PCB version
Version 6 of the SDR Design
Parts:
- C14, C9: value 7.5n -> 6.8n
- C16, C17: value 14p -> 1n
- R10, R9: value 160 -> 51
- R7, R8: value 51k -> 5.1k
Other:
- note added: "Cadyn Maddocks & Taylor Smith SDR Receiver Electronics II V6"
- note added: "Multiple Feedback Lowpass Filter & Amplifier 25 V/V with Cutoff Frequency of approx 100kHz"
- note removed: "Cadyn Maddocks & Taylor Smith SDR Receiver Electronics II V4"
- note removed: "Multiple Feedback Lowpass Filter & Amplifier 1000 V/V with Cutoff Frequency of approx 100kHz"
Changed lines of the file:
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@@
     (stroke (width 0) (type default) (color 0 0 0 0))
   )
-  (text "Multiple Feedback Lowpass Filter & Amplifier\n1000 V/V with Cutoff Frequency of approx 100kHz\n"
+  (text "Multiple Feedback Lowpass Filter & Amplifier\n25 V/V with Cutoff Frequency of approx 100kHz\n"
     (at 175.26 19.05 0)
     (effects (font (size 1.27 1.27)) (justify left bottom))
@@
     (effects (font (size 1.27 1.27)) (justify left bottom))
   )
-  (text "Cadyn Maddocks & Taylor Smith\nSDR Receiver\nElectronics II\nV4\n"
+  (text "Cadyn Maddocks & Taylor Smith\nSDR Receiver\nElectronics II\nV6\n"
     (at 21.59 27.94 0)
     (effects (font (size 1.27 1.27)) (justify left bottom))
@@
       (effects (font (size 1.27 1.27)) (justify left))
     )
-    (property "Value" "7.5n" (id 1) (at 189.23 59.6962 0)
+    (property "Value" "6.8n" (id 1) (at 189.23 59.6962 0)
       (effects (font (size 1.27 1.27)) (justify left))
     )
@@
     (in_bom yes) (on_board yes) (fields_autoplaced)
     (property "Reference" "R7" (id 0) (at 193.04 76.2 90))
-    (property "Value" "51k" (id 1) (at 193.04 78.74 90))
+    (property "Value" "5.1k" (id 1) (at 193.04 78.74 90))
     (property "Footprint" "Resistor_SMD:R_0805_2012Metric" (id 2) (at 193.04 82.55 0)
       (effects (font (size 1.27 1.27)) hide)
@@
       (effects (font (size 1.27 1.27)) (justify left))
     )
-    (property "Value" "14p" (id 1) (at 204.47 31.7562 0)
+    (property "Value" "1n" (id 1) (at 204.47 31.7562 0)
       (effects (font (size 1.27 1.27)) (justify left))
     )
@@
       (effects (font (size 1.27 1.27)) (justify left))
     )
-    (property "Value" "14p" (id 1) (at 204.47 77.4762 0)
+    (property "Value" "1n" (id 1) (at 204.47 77.4762 0)
       (effects (font (size 1.27 1.27)) (justify left))
     )
@@
     (pin "1")
   )
-  (symbol (lib_id "power:+3.3V") (at 78.74 111.76 0) (unit 1)
-    (in_bom yes) (on_board yes) (fields_autoplaced)
-    (property "Reference" "#PWR05" (id 0) (at 78.74 115.57 0)
-      (effects (font (size 1.27 1.27)) hide)
-    )
-    (property "Value" "+3.3V" (id 1) (at 78.74 106.68 0))
+  (symbol (lib_id "power:+3.3V") (at 78.74 111.76 270) (unit 1)
+    (in_bom yes) (on_board yes) (fields_autoplaced)
+    (property "Reference" "#PWR05" (id 0) (at 74.93 111.76 0)
+      (effects (font (size 1.27 1.27)) hide)
+    )
+    (property "Value" "+3.3V" (id 1) (at 82.55 111.7599 90)
+      (effects (font (size 1.27 1.27)) (justify left))
+    )
     (property "Footprint" "" (id 2) (at 78.74 111.76 0)
       (effects (font (size 1.27 1.27)) hide)
@@
       (effects (font (size 1.27 1.27)) (justify left))
     )
-    (property "Value" "7.5n" (id 1) (at 189.23 52.0762 0)
+    (property "Value" "6.8n" (id 1) (at 189.23 52.0762 0)
       (effects (font (size 1.27 1.27)) (justify left))
     )
@@
     (in_bom yes) (on_board yes) (fields_autoplaced)
     (property "Reference" "R8" (id 0) (at 195.58 20.32 90))
-    (property "Value" "51k" (id 1) (at 195.58 22.86 90))
+    (property "Value" "5.1k" (id 1) (at 195.58 22.86 90))
     (property "Footprint" "Resistor_SMD:R_0805_2012Metric" (id 2) (at 195.58 26.67 0)
       (effects (font (size 1.27 1.27)) hide)
@@
     (in_bom yes) (on_board yes)
     (property "Reference" "R10" (id 0) (at 196.85 64.77 90))
-    (property "Value" "160" (id 1) (at 196.85 67.31 90))
+    (property "Value" "51" (id 1) (at 196.85 67.31 90))
     (property "Footprint" "Resistor_SMD:R_0805_2012Metric" (id 2) (at 196.85 69.85 0)
       (effects (font (size 1.27 1.27)) hide)
@@
     (in_bom yes) (on_board yes) (fields_autoplaced)
     (property "Reference" "R9" (id 0) (at 195.58 29.21 90))
-    (property "Value" "160" (id 1) (at 195.58 31.75 90))
+    (property "Value" "51" (id 1) (at 195.58 31.75 90))
     (property "Footprint" "Resistor_SMD:R_0805_2012Metric" (id 2) (at 195.58 35.56 0)
       (effects (font (size 1.27 1.27)) hide)
@@
     )
     (path "/e74cb884-ae67-437b-a63e-c252033ca7f2"
-      (reference "C9") (unit 1) (value "7.5n") (footprint "Capacitor_SMD:C_0805_2012Metric")
+      (reference "C9") (unit 1) (value "6.8n") (footprint "Capacitor_SMD:C_0805_2012Metric")
     )
     (path "/33f197c7-472d-407b-a7c3-ca5bf645861f"
@@
     )
     (path "/113ef254-820a-43ee-81cd-2b01c043d894"
-      (reference "C14") (unit 1) (value "7.5n") (footprint "Capacitor_SMD:C_0805_2012Metric")
+      (reference "C14") (unit 1) (value "6.8n") (footprint "Capacitor_SMD:C_0805_2012Metric")
     )
     (path "/12a4a4ec-1bc7-46d4-a729-c41e56dd799d"
@@
     )
     (path "/7ca7273b-db13-441c-8aa4-5d5d29a90e38"
-      (reference "C16") (unit 1) (value "14p") (footprint "Capacitor_SMD:C_0805_2012Metric")
+      (reference "C16") (unit 1) (value "1n") (footprint "Capacitor_SMD:C_0805_2012Metric")
     )
     (path "/92072820-a231-4001-aa0b-fa9aee3d6275"
-      (reference "C17") (unit 1) (value "14p") (footprint "Capacitor_SMD:C_0805_2012Metric")
+      (reference "C17") (unit 1) (value "1n") (footprint "Capacitor_SMD:C_0805_2012Metric")
     )
     (path "/07524787-cdb6-4115-868a-4775882d4f0c"
@@
     )
     (path "/4cb98030-e11d-46ec-ace2-24b8060477eb"
-      (reference "R7") (unit 1) (value "51k") (footprint "Resistor_SMD:R_0805_2012Metric")
+      (reference "R7") (unit 1) (value "5.1k") (footprint "Resistor_SMD:R_0805_2012Metric")
     )
     (path "/f02277ed-a9de-4a94-9a7a-bd1104f6b9ca"
-      (reference "R8") (unit 1) (value "51k") (footprint "Resistor_SMD:R_0805_2012Metric")
+      (reference "R8") (unit 1) (value "5.1k") (footprint "Resistor_SMD:R_0805_2012Metric")
     )
     (path "/ffd130c3-85b2-4c7b-9ad6-0a05ac6435fc"
-      (reference "R9") (unit 1) (value "160") (footprint "Resistor_SMD:R_0805_2012Metric")
+      (reference "R9") (unit 1) (value "51") (footprint "Resistor_SMD:R_0805_2012Metric")
     )
     (path "/f11b3e3a-7b08-49d8-b4b1-92030ffe70c2"
-      (reference "R10") (unit 1) (value "160") (footprint "Resistor_SMD:R_0805_2012Metric")
+      (reference "R10") (unit 1) (value "51") (footprint "Resistor_SMD:R_0805_2012Metric")
     )
     (path "/59020215-584d-45e3-9399-bfe29ae3a841"

Commit message: Block Diagram Upload
Other:
- note added: "Multiple Feedback Lowpass Filter & Amplifier 25 V/V with Cutoff Frequency of approx 60kHz"
- note removed: "Multiple Feedback Lowpass Filter & Amplifier 25 V/V with Cutoff Frequency of approx 100kHz"
Changed lines of the file:
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@@
     (stroke (width 0) (type default) (color 0 0 0 0))
   )
-  (text "Multiple Feedback Lowpass Filter & Amplifier\n25 V/V with Cutoff Frequency of approx 100kHz\n"
+  (text "Multiple Feedback Lowpass Filter & Amplifier\n25 V/V with Cutoff Frequency of approx 60kHz\n"
     (at 175.26 19.05 0)
     (effects (font (size 1.27 1.27)) (justify left bottom))

Commit message: Added Bandpass filter simulation
Parts:
- C3: value 130pF -> (none); footprint Capacitor_SMD:C_0805_2012Metric -> (none)
- C5: value 2.2nF -> (none)
- C7: value 130pF -> (none)
- L1, L3: value 2.7uH -> (none)
- L2: value 180nH -> (none)
Changed lines of the file:
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@@
     (in_bom yes) (on_board yes) (fields_autoplaced)
     (property "Reference" "L3" (id 0) (at 81.28 50.8 90))
-    (property "Value" "2.7uH" (id 1) (at 81.28 53.34 90))
+    (property "Value" "" (id 1) (at 81.28 53.34 90))
     (property "Footprint" "Inductor_THT:L_Toroid_Vertical_L10.0mm_W5.0mm_P5.08mm" (id 2) (at 81.28 57.15 0)
       (effects (font (size 1.27 1.27)) hide)
@@
     (in_bom yes) (on_board yes) (fields_autoplaced)
     (property "Reference" "C7" (id 0) (at 74.9363 50.8 90))
-    (property "Value" "130pF" (id 1) (at 74.9363 53.34 90))
+    (property "Value" "" (id 1) (at 74.9363 53.34 90))
     (property "Footprint" "Capacitor_SMD:C_0805_2012Metric" (id 2) (at 74.93 57.15 0)
       (effects (font (size 1.27 1.27)) hide)
@@
     (in_bom yes) (on_board yes) (fields_autoplaced)
     (property "Reference" "C3" (id 0) (at 39.3636 50.8 90))
-    (property "Value" "130pF" (id 1) (at 39.3636 53.34 90))
-    (property "Footprint" "Capacitor_SMD:C_0805_2012Metric" (id 2) (at 39.37 57.15 0)
+    (property "Value" "" (id 1) (at 39.3636 53.34 90))
+    (property "Footprint" "" (id 2) (at 39.37 57.15 0)
       (effects (font (size 1.27 1.27)) hide)
     )
@@
       (effects (font (size 1.27 1.27)) (justify left))
     )
-    (property "Value" "2.2nF" (id 1) (at 58.42 64.7762 0)
+    (property "Value" "" (id 1) (at 58.42 64.7762 0)
       (effects (font (size 1.27 1.27)) (justify left))
     )
@@
       (effects (font (size 1.27 1.27)) (justify left))
     )
-    (property "Value" "180nH" (id 1) (at 69.85 64.7699 0)
+    (property "Value" "" (id 1) (at 69.85 64.7699 0)
       (effects (font (size 1.27 1.27)) (justify left))
     )
@@
     (in_bom yes) (on_board yes) (fields_autoplaced)
     (property "Reference" "L1" (id 0) (at 45.72 50.8 90))
-    (property "Value" "2.7uH" (id 1) (at 45.72 53.34 90))
+    (property "Value" "" (id 1) (at 45.72 53.34 90))
     (property "Footprint" "Inductor_THT:L_Toroid_Vertical_L10.0mm_W5.0mm_P5.08mm" (id 2) (at 45.72 57.15 0)
       (effects (font (size 1.27 1.27)) hide)
@@
     )
     (path "/2590172d-4ae2-40ab-a929-249ba6bbda91"
-      (reference "C3") (unit 1) (value "130pF") (footprint "Capacitor_SMD:C_0805_2012Metric")
+      (reference "C3") (unit 1) (value "180pF") (footprint "Capacitor_SMD:C_0805_2012Metric")
     )
     (path "/3f47af1e-9f6e-42de-b693-8f75c1b06bd5"
@@
     )
     (path "/847820eb-ddb9-4714-9f93-4cf047f6a900"
-      (reference "C5") (unit 1) (value "2.2nF") (footprint "Capacitor_SMD:C_0805_2012Metric")
+      (reference "C5") (unit 1) (value "1.3nF") (footprint "Capacitor_SMD:C_0805_2012Metric")
     )
     (path "/d946fa37-827d-4a94-82df-218df4f30c3d"
@@
     )
     (path "/20943f1c-cff2-4afe-969d-6ed0d9cb647b"
-      (reference "C7") (unit 1) (value "130pF") (footprint "Capacitor_SMD:C_0805_2012Metric")
+      (reference "C7") (unit 1) (value "180pF") (footprint "Capacitor_SMD:C_0805_2012Metric")
     )
     (path "/f1bbc74e-8bcb-4555-8b76-efdc59bd3042"
@@
     )
     (path "/d281e302-963d-4e62-8db4-039301c9dfc3"
-      (reference "L1") (unit 1) (value "2.7uH") (footprint "Inductor_THT:L_Toroid_Vertical_L10.0mm_W5.0mm_P5.08mm")
+      (reference "L1") (unit 1) (value "1.6uH") (footprint "Inductor_THT:L_Toroid_Vertical_L10.0mm_W5.0mm_P5.08mm")
     )
     (path "/cca85874-6ab0-4e57-ad06-f91b8f453cfa"
-      (reference "L2") (unit 1) (value "180nH") (footprint "Inductor_THT:L_Toroid_Vertical_L10.0mm_W5.0mm_P5.08mm")
+      (reference "L2") (unit 1) (value "240nH") (footprint "Inductor_THT:L_Toroid_Vertical_L10.0mm_W5.0mm_P5.08mm")
     )
     (path "/0b1b5880-6d40-43fb-847e-8ebd98ff1a7d"
-      (reference "L3") (unit 1) (value "2.7uH") (footprint "Inductor_THT:L_Toroid_Vertical_L10.0mm_W5.0mm_P5.08mm")
+      (reference "L3") (unit 1) (value "1.6uH") (footprint "Inductor_THT:L_Toroid_Vertical_L10.0mm_W5.0mm_P5.08mm")
     )
     (path "/c7098508-2196-420a-91a4-04f1a230c0a8"
